File: attiny416_breakout/pcb/attiny416_breakout.kicad_sch (KiCad schematic)
At the start: 9 parts, among them J1 PROG, J2 5V, J3 GND, J4 Conn_01x10, J5 Conn_01x10, U1 ATtiny416-S

Commit message: create breakout
Parts:
- C1: footprint Capacitor_SMD:C_0603_1608Metric_Pad1.08x0.95mm_HandSolder -> Capacitor_THT:C_Rect_L7.0mm_W2.0mm_P5.00mm
- D1: footprint LED_SMD:LED_0805_2012Metric_Pad1.15x1.40mm_HandSolder -> LED_THT:LED_D5.0mm
Connections:
- net +5V: now also J4.1 (Pin_1)
- net GND: now also J5.1 (Pin_1)
- no-connect marks 3 -> 1
Changed lines of the file:
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@@
+		(color 0 0 0 0)
+	)
+	(junction
+		(at 66.04 90.17)
+		(diameter 0)
 		(color 0 0 0 0)
 	)
@@
 		(at 85.09 110.49)
 	)
-	(no_connect
-		(at 85.09 100.33)
-	)
-	(no_connect
-		(at 63.5 100.33)
-	)
 	(wire
 		(pts
@@
 	(wire
 		(pts
+			(xy 80.01 100.33) (xy 80.01 90.17)
+		)
+		(stroke
+			(width 0)
+			(type default)
+		)
+	)
+	(wire
+		(pts
 			(xy 153.67 66.04) (xy 153.67 68.58)
 		)
@@
 	(wire
 		(pts
+			(xy 66.04 100.33) (xy 66.04 90.17)
+		)
+		(stroke
+			(width 0)
+			(type default)
+		)
+	)
+	(wire
+		(pts
 			(xy 80.01 107.95) (xy 85.09 107.95)
 		)
@@
 	(wire
 		(pts
+			(xy 85.09 100.33) (xy 80.01 100.33)
+		)
+		(stroke
+			(width 0)
+			(type default)
+		)
+	)
+	(wire
+		(pts
 			(xy 161.29 110.49) (xy 156.21 110.49)
 		)
@@
 	(wire
 		(pts
+			(xy 80.01 90.17) (xy 82.55 90.17)
+		)
+		(stroke
+			(width 0)
+			(type default)
+		)
+	)
+	(wire
+		(pts
 			(xy 214.63 50.8) (xy 212.09 50.8)
 		)
@@
 		(pts
 			(xy 212.09 50.8) (xy 212.09 53.34)
+		)
+		(stroke
+			(width 0)
+			(type default)
+		)
+	)
+	(wire
+		(pts
+			(xy 63.5 100.33) (xy 66.04 100.33)
 		)
 		(stroke
@@
 			)
 		)
-		(property "Footprint" "LED_SMD:LED_0805_2012Metric_Pad1.15x1.40mm_HandSolder"
+		(property "Footprint" "LED_THT:LED_D5.0mm"
 			(at 181.61 113.03 0)
 			(effects
@@
 			)
 		)
-		(property "Footprint" "Capacitor_SMD:C_0603_1608Metric_Pad1.08x0.95mm_HandSolder"
+		(property "Footprint" "Capacitor_THT:C_Rect_L7.0mm_W2.0mm_P5.00mm"
 			(at 151.13 65.0748 0)
 			(effects

Commit message: breakout UPDI
Connections:
- net UPDI: now also J5.5 (Pin_5)
- no-connect marks 1 -> 0
Changed lines of the file:
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@@
 		(color 0 0 0 0)
 	)
-	(no_connect
-		(at 85.09 110.49)
-	)
 	(wire
 		(pts
@@
 		(pts
 			(xy 161.29 105.41) (xy 156.21 105.41)
+		)
+		(stroke
+			(width 0)
+			(type default)
+		)
+	)
+	(wire
+		(pts
+			(xy 80.01 110.49) (xy 85.09 110.49)
 		)
 		(stroke
@@
 		)
 	)
+	(label "UPDI"
+		(at 80.01 110.49 180)
+		(fields_autoplaced yes)
+		(effects
+			(font
+				(size 1.27 1.27)
+			)
+			(justify right bottom)
+		)
+	)
