File: xtal_tester/pcb/xtal_tester.kicad_pcb (KiCad board)
At the start: 2 copper layers, 48.5 x 35.6 mm, 20 parts, among them J1 Conn_01x04, J2 Conn_01x04, J3 Conn_01x04, Q1 Q_NPN_ECB, Q2 Q_NPN_ECB, Y1 Crystal

Commit message: change xtal footprint to pin header
Parts:
- removed Y1: Crystal, Crystal:Crystal_HC18-U_Vertical
- added J4: xtal, Connector_PinHeader_2.54mm:PinHeader_1x03_P2.54mm_Vertical, F.Cu at (117.1, 102.1)
Routing:
- net GND: track 59.0 -> 61.0 mm
- net Net-(J4-Pin_1): track 15.2 -> 15.9 mm
