File: opamp_motor_position/pcb/opamp_motor_position.kicad_sch (KiCad schematic)
At the start: 21 parts, among them J1 Conn_01x02, J2 Conn_01x02, J3 Conn_01x02, J4 Conn_01x02, M1 Motor_DC, Q1 Q_NPN_BCE, Q2 Q_PNP_BCE, U1 LM358

Commit message: Update opamp_motor_position.kicad_sch
Parts:
- removed Q1: Q_NPN_BCE, symbol Device:Q_NPN_BCE
- removed Q2: Q_PNP_BCE, symbol Device:Q_PNP_BCE
- added JP1: Vset Select, Connector_PinHeader_2.54mm:PinHeader_1x03_P2.54mm_Vertical, symbol Jumper:Jumper_3_Bridged12
- added Q1: 2N6037, Package_TO_SOT_THT:TO-126-3_Vertical, symbol Device:Q_NPN_ECB
- added Q2: 2N6036, Package_TO_SOT_THT:TO-126-3_Vertical, symbol Device:Q_PNP_ECB
- added RV1: 100k, Potentiometer_THT:Potentiometer_Alps_RK163_Single_Horizontal, symbol Device:R_Potentiometer
- M1: footprint (none) -> TerminalBlock_Altech:Altech_AK100_1x02_P5.00mm
- renumbered H4 to H3, H3 to H4, J4 to J1, J1 to J2, J2 to J3, J3 to J4, RV1 to RV2, RV2 to RV3
Connections:
- net +12V: now also Q1.2 (C), RV1.1
- net -12V: now also Q2.2 (C), RV1.3
- net Vset: now also JP1.2 (C); no longer J1.1 (Pin_1), J1.2 (Pin_2)
- net at U1.7: now also Q1.3 (B), Q2.3 (B)
- net at M1.1 (+), U1.6 (-): now also Q1.1 (E), Q2.1 (E)
- new net: JP1.1 (A), RV1.2
- new net Vext: J1.1 (Pin_1), J1.2 (Pin_2), JP1.3 (B)
Other:
- moved on the sheet: J1

Commit message: pcb layout 1
Parts:
- H1, H2, H3, H4: footprint MountingHole:MountingHole_3.2mm_M3_Pad_Via -> MountingHole:MountingHole_3.2mm_M3_Pad_TopBottom
Connections:
- net +12V: now also RV3.3; no longer RV3.1
- net -12V: now also RV3.1; no longer RV3.3
- net at R3.1, RV2.2, U1.1: now also RV2.1; no longer RV2.3
- net at R1.2, R2.2, U1.2 (-): now also RV2.3; no longer RV2.1
Other:
- title: Opamp Closed Loop Position Control -> Opamp Motor Position Control
- moved on the sheet: RV2
Changed lines of the file:
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@@
 	(paper "A")
 	(title_block
-		(title "Opamp Closed Loop Position Control")
+		(title "Opamp Motor Position Control")
+		(date "2024-05-09")
 		(company "Perry Leumas")
 	)
@@
 			)
 		)
-		(property "Footprint" "MountingHole:MountingHole_3.2mm_M3_Pad_Via"
+		(property "Footprint" "MountingHole:MountingHole_3.2mm_M3_Pad_TopBottom"
 			(at 127 127 0)
 			(effects
@@
 			)
 		)
-		(property "Footprint" "MountingHole:MountingHole_3.2mm_M3_Pad_Via"
+		(property "Footprint" "MountingHole:MountingHole_3.2mm_M3_Pad_TopBottom"
 			(at 127 114.3 0)
 			(effects
@@
 		(lib_id "Device:R_Potentiometer")
 		(at 193.04 68.58 0)
+		(mirror x)
 		(unit 1)
 		(exclude_from_sim no)
@@
 	(symbol
 		(lib_id "Device:R_Potentiometer")
-		(at 88.9 41.91 90)
+		(at 88.9 41.91 270)
+		(mirror x)
 		(unit 1)
 		(exclude_from_sim no)
@@
 			)
 		)
-		(property "Footprint" "MountingHole:MountingHole_3.2mm_M3_Pad_Via"
+		(property "Footprint" "MountingHole:MountingHole_3.2mm_M3_Pad_TopBottom"
 			(at 146.05 114.3 0)
 			(effects
@@
 			)
 		)
-		(property "Footprint" "MountingHole:MountingHole_3.2mm_M3_Pad_Via"
+		(property "Footprint" "MountingHole:MountingHole_3.2mm_M3_Pad_TopBottom"
 			(at 146.05 127 0)
 			(effects
