File: opamp_motor_position/pcb/opamp_motor_position.kicad_pcb (KiCad board)
At the start: 2 copper layers, 75.1 x 51.3 mm, 23 parts, among them J1 Conn_01x02, J2 Conn_01x02, J3 Conn_01x02, J4 Conn_01x02, M1 Motor_DC, Q1 2N6037, Q2 2N6036, U1 LM358

Commit message: pcb gcode
Parts:
- moved Q2 8.19 mm to (126.0, 81.8), turned to -90 degrees
- moved Q1 5.79 mm to (119.7, 81.8)
- moved M1 4.95 mm to (135.1, 83.8)
- moved C3 1.30 mm to (112.4, 93.1)
- moved C4 1.30 mm to (128.8, 95.7)
Routing:
- net +12V: track 160.7 -> 49.3 mm
- net -12V: track 84.4 -> 18.6 mm, vias 0 -> 2
- net Net-(M1-+): track 70.3 -> 28.1 mm
- net GND: track 19.0 -> 3.53 mm
- net Net-(U1B-+): track 29.9 -> 22.4 mm, vias 0 -> 2
- net Net-(Q1-B): track 23.2 -> 29.5 mm
