File: XL1410E1/xl1410e1.kicad_pcb (KiCad board)
At the start: 2 copper layers, 39 x 42.5 mm, 18 parts, among them J1 Conn_01x04, J2 Conn_01x04, J3 Conn_01x04, J4 Conn_01x04, U1 XL1410

Commit message: output ibom
Parts:
- R1: value 2k -> 2k2
- R2: value 6k2 -> 6k8
Changed lines of the file:
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@@
 		(tags "Through hole pin header THT 1x04 2.54mm single row")
 		(property "Reference" "J1"
-			(at 0 -2.33 360)
+			(at 0 -2.33 0)
 			(layer "F.SilkS")
 			(effects
@@
 		)
 		(property "Value" "Conn_01x04"
-			(at 0 9.95 360)
+			(at 0 9.95 0)
 			(layer "F.Fab")
 			(effects
@@
 			)
 		)
-		(property "Value" "6k2"
+		(property "Value" "6k8"
 			(at 5.08 2.37 0)
 			(layer "F.Fab")
@@
 		)
 		(fp_text user "${REFERENCE}"
-			(at 0 3.81 360)
+			(at 0 3.81 0)
 			(layer "F.Fab")
 			(effects
@@
 		)
 		(fp_text user "${REFERENCE}"
-			(at 0 3.81 360)
+			(at 0 3.81 0)
 			(layer "F.Fab")
 			(effects
@@
 			)
 		)
-		(property "Value" "2k"
+		(property "Value" "2k2"
 			(at 5.08 2.37 90)
 			(layer "F.Fab")
@@
 		)
 		(fp_text user "${REFERENCE}"
-			(at 0 3.81 360)
+			(at 0 3.81 0)
 			(layer "F.Fab")
 			(effects
@@
 	)
 	(zone
-		(net 4)
-		(net_name "Net-(U1-FB)")
+		(net 6)
+		(net_name "Net-(U1-EN)")
 		(layer "B.Cu")
 		(name "$teardrop_padvia$")
 		(hatch full 0.1)
-		(priority 30003)
+		(priority 30004)
 		(attr
 			(teardrop
@@
 		(polygon
 			(pts
-				(xy 142.86 78.39) (xy 142.06 78.39) (xy 141.720896 79.683853) (xy 142.46 79.991) (xy 143.199104 79.683853)
+				(xy 143.63 65.08) (xy 143.63 64.28) (xy 142.336147 63.940896) (xy 142.029 64.68) (xy 142.336147 65.419104)
 			)
 		)
@@
 		(name "$teardrop_padvia$")
 		(hatch full 0.1)
-		(priority 30002)
+		(priority 30001)
 		(attr
 			(teardrop
@@
 		(polygon
 			(pts
-				(xy 144.07 77.83) (xy 144.07 77.03) (xy 142.776147 76.690896) (xy 142.469 77.43) (xy 142.776147 78.169104)
+				(xy 142.86 78.39) (xy 142.06 78.39) (xy 141.720896 79.683853) (xy 142.46 79.991) (xy 143.199104 79.683853)
 			)
 		)
 	)
 	(zone
-		(net 6)
-		(net_name "Net-(U1-EN)")
+		(net 4)
+		(net_name "Net-(U1-FB)")
 		(layer "B.Cu")
 		(name "$teardrop_padvia$")
 		(hatch full 0.1)
-		(priority 30004)
+		(priority 30000)
 		(attr
 			(teardrop
@@
 		(polygon
 			(pts
-				(xy 143.63 65.08) (xy 143.63 64.28) (xy 142.336147 63.940896) (xy 142.029 64.68) (xy 142.336147 65.419104)
+				(xy 144.07 77.83) (xy 144.07 77.03) (xy 142.776147 76.690896) (xy 142.469 77.43) (xy 142.776147 78.169104)
 			)
 		)
@@
 	)
 	(zone
-		(net 3)
-		(net_name "+5V")
-		(layer "B.Cu")
-		(hatch edge 0.5)
-		(priority 3)
-		(connect_pads
-			(clearance 0.5)
-		)
-		(min_thickness 0.25)
-		(filled_areas_thickness no)
-		(fill yes
-			(thermal_gap 0.5)
-			(thermal_bridge_width 0.8)
-		)
-		(polygon
-			(pts
-				(xy 141.41 85.14) (xy 141.41 81.54) (xy 150.36 81.54) (xy 150.36 77.71) (xy 162.62 77.71) (xy 162.62 85.14)
-			)
-		)
-	)
-	(zone
 		(net 4)
 		(net_name "Net-(U1-FB)")
@@
 		(name "$teardrop_padvia$")
 		(hatch full 0.1)
-		(priority 30006)
+		(priority 30002)
 		(attr
 			(teardrop
@@
 			)
 		)
+	)
+	(zone
+		(net 3)
+		(net_name "+5V")
+		(layer "B.Cu")
+		(hatch edge 0.5)
+		(priority 3)
+		(connect_pads
+			(clearance 0.5)
+		)
+		(min_thickness 0.25)
+		(filled_areas_thickness no)
+		(fill yes
+			(thermal_gap 0.5)
+			(thermal_bridge_width 0.8)
+		)
+		(polygon
+			(pts
+				(xy 141.41 85.14) (xy 141.41 81.54) (xy 150.36 81.54) (xy 150.36 77.71) (xy 162.62 77.71) (xy 162.62 85.14)
+			)
+		)
