File: lcd_3digit/pcb/lcd_3digit.kicad_sch (KiCad schematic)
At the start: 10 parts, among them J1 Conn_01x03, U1 ATtiny416-S

Commit message: create test pcb
Parts:
- removed C1: C, Capacitor_THT:C_Rect_L7.0mm_W2.0mm_P5.00mm, symbol Device:C
- removed J1: Conn_01x03, symbol Connector_Generic:Conn_01x03
- removed R1, R2, R3, R4, R5, R6: R, symbol Device:R
- removed U1: ATtiny416-S, Package_SO:SOIC-20W_7.5x12.8mm_P1.27mm, symbol MCU_Microchip_ATtiny:ATtiny416-S
- added J1, J2: Conn_01x05, Connector_PinHeader_2.54mm:PinHeader_1x05_P2.54mm_Vertical, symbol Connector_Generic:Conn_01x05
- D1: footprint (none) -> pl_LCD:LCD_3_Digit_10p
Connections:
- net at D1.2: now also J2.2 (Pin_2)
- net at D1.1: now also J2.1 (Pin_1)
- net at D1.3: now also J2.3 (Pin_3)
- net at D1.4: now also J2.4 (Pin_4)
- net at D1.5: now also J2.5 (Pin_5)
- net at D1.6: now also J1.5 (Pin_5)
- net COM1: no longer names the net of D1.10 (COM1)
- net COM1: now also J1.1 (Pin_1)
- net COM2: no longer names the net of D1.9 (COM2)
- net COM2: now also J1.2 (Pin_2)
- net COM3: no longer names the net of D1.8 (COM3)
- net COM3: now also J1.3 (Pin_3)
- net COM4: no longer names the net of D1.7 (COM4)
- net COM4: now also J1.4 (Pin_4)
Other:
- moved on the sheet: D1
